File: hw/guitarif/guitarif.kicad_pcb (KiCad board)
At the start: 2 copper layers, 43 x 42.4 mm, 28 parts, among them J1 Barrel_Jack_Switch, J2 Barrel_Jack_Switch, J3 Conn_01x04, U1 Opamp_Dual_Generic

Commit message: fixed schematic bug in potentiometer
Parts:
- removed REF***: OSHW-Logo2_7.3x6mm_SilkScreen, Symbols:OSHW-Logo2_7.3x6mm_SilkScreen
Connections:
- RV1 pad 2: Net-(C8-Pad2) -> Net-(R6-Pad1)
- RV1 pad 3: Net-(R6-Pad1) -> (no net)
Routing:
- net Net-(C8-Pad2): track 18.5 -> 13.6 mm
Other:
- board text added: "Guitar IF Ver 0.2 By H.Kim Dec, 2018"
- board text removed: "Guitar IF Ver 0.1 By H.Kim Dec, 2018"
