File: hw/guitarif/guitarif.sch (KiCad schematic (older format))
At the start: 27 parts, among them J1 Barrel_Jack_Switch, J2 Barrel_Jack_Switch, J3 Conn_01x04, U1 Opamp_Dual_Generic

Commit message: fixed schematic bug in potentiometer
Connections:
- no-connect marks 0 -> 1
Changed lines of the file:
@@
 Wire Wire Line
 	5550 850  5900 850
-Wire Wire Line
-	5550 850  5550 1000
-Wire Wire Line
-	5550 1250 5150 1250
 Connection ~ 5550 1250
-Wire Wire Line
-	5000 1100 5000 1000
-Wire Wire Line
-	5000 1000 5550 1000
-Connection ~ 5550 1000
-Wire Wire Line
-	5550 1000 5550 1250
 $Comp
 L Device:R R6
@@
 	0    1    1    0
 $EndComp
-Wire Wire Line
-	4850 1250 4500 1250
 $Comp
 L Device:CP C3
@@
 Wire Wire Line
 	4850 5600 5200 5600
+Wire Wire Line
+	5550 850  5550 1250
+Wire Wire Line
+	5550 1250 5150 1250
+Wire Wire Line
+	4500 1250 4650 1250
+Wire Wire Line
+	4650 1250 4650 1000
+Wire Wire Line
+	4650 1000 5000 1000
+Wire Wire Line
+	5000 1000 5000 1100
+NoConn ~ 4850 1250
 $EndSCHEMATC
